Commit message: fixing wheel slippage (WIP) and orientation issues with rviz

File: ros2/description/urdf/terrence.urdf.xacro (robot description, xacro)
@@ -38,5 +38,5 @@
   </link>
   <joint name="Baseplate_joint" type="fixed">
-    <origin xyz="0 0 0" rpy="${pi/2} 0 0" />
+    <origin xyz="0.136145 0 0" rpy="${pi/2} 0 ${pi/2}" />
     <parent link="base_link" />
     <child link="Base" />
@@ -62,7 +62,8 @@
     </visual>
     <collision>
-      <origin xyz="0 0 0" rpy="0 0 0" />
-      <geometry>
-        <mesh filename="file://$(find description)/meshes/DriverWheel.STL" />
+      <origin xyz="-0.030264 6.665E-05 1.2263E-10" rpy="0 0 0" />
+      <geometry>
+        <!-- <mesh filename="file://$(find description)/meshes/DriverWheel.STL" /> -->
+        <sphere radius="0.0397"/>
       </geometry>
     </collision>
@@ -78,6 +79,10 @@
   <gazebo reference="DriverWheel">
     <material>Gazebo/Blue</material>
+      <!-- <mu1 value="0.001"/>
+      <mu2 value="0.001"/> -->
       <mu1 value="0.001"/>
       <mu2 value="0.001"/>
+      <!-- <kp value="10000000.0" />
+      <kd value="1.0" /> -->
   </gazebo>
   <link name="DriverSprocket">
@@ -98,7 +103,8 @@
     </visual>
     <collision>
-      <origin xyz="0 0 0" rpy="0 0 0" />
-      <geometry>
-        <mesh filename="file://$(find description)/meshes/DriverSprocket.STL" />
+      <origin xyz="0.0097746 -3.5292E-09 -5.2457E-08" rpy="0 0 0" />
+      <geometry>
+        <!-- <mesh filename="file://$(find description)/meshes/DriverSprocket.STL" /> -->
+        <sphere radius="0.0397"/>
       </geometry>
     </collision>
@@ -113,4 +119,6 @@
   <gazebo reference="DriverSprocket">
     <material>Gazebo/Blue</material>
+      <mu1 value="1.0"/>
+      <mu2 value="1.0"/>
   </gazebo>
   <link name="PassWheel">
@@ -131,7 +139,8 @@
     </visual>
     <collision>
-      <origin xyz="0 0 0" rpy="0 0 0" />
-      <geometry>
-        <mesh filename="file://$(find description)/meshes/PassWheel.STL" />
+      <origin xyz="0.020612 8.4006E-05 -0.00023239" rpy="0 0 0" />
+      <geometry>
+        <!-- <mesh filename="file://$(find description)/meshes/PassWheel.STL" /> -->
+        <sphere radius="0.0397"/>
       </geometry>
     </collision>
@@ -167,7 +176,8 @@
     </visual>
     <collision>
-      <origin xyz="0 0 0" rpy="0 0 0" />
-      <geometry>
-        <mesh filename="file://$(find description)/meshes/PassSprocket.STL" />
+      <origin xyz="-0.0056813 -3.6211E-09 -5.2434E-08" rpy="0 0 0" />
+      <geometry>
+        <!-- <mesh filename="file://$(find description)/meshes/PassSprocket.STL" /> -->
+        <sphere radius="0.0397"/>
       </geometry>
     </collision>
@@ -182,4 +192,6 @@
   <gazebo reference="PassSprocket">
     <material>Gazebo/Blue</material>
+      <mu1 value="1.0"/>
+      <mu2 value="1.0"/>
   </gazebo>
   <link name="Loader">
