Commit message: fixed urdf package references

File: ros2/description/urdf/ros2_control.xacro (robot description, xacro)
@@ -79,5 +79,5 @@
     <gazebo>
         <plugin name="gz_ros2_control::GazeboSimROS2ControlPlugin" filename="libgz_ros2_control-system.so">
-            <parameters>$(find terrence_2)/config/my_controllers.yaml</parameters>
+            <parameters>$(find control)/config/controllers.yaml</parameters>
         </plugin>
     </gazebo>

File: ros2/description/urdf/terrence.urdf.xacro (robot description, xacro)
@@ -26,5 +26,5 @@
       <origin xyz="0 0 0" rpy="0 0 0" />
       <geometry>
-        <mesh filename="file://$(find terrence_2)/description/meshes/Base.STL" />
+        <mesh filename="file://$(find description)/meshes/Base.STL" />
       </geometry>
       <material name="">
@@ -35,5 +35,5 @@
       <origin xyz="0 0 0" rpy="0 0 0" />
       <geometry>
-        <mesh filename="file://$(find terrence_2)/description/meshes/Base.STL" />
+        <mesh filename="file://$(find description)/meshes/Base.STL" />
       </geometry>
     </collision>
@@ -57,14 +57,14 @@
       <origin xyz="0 0 0" rpy="0 0 0" />
       <geometry>
-        <mesh filename="file://$(find terrence_2)/description/meshes/DriverWheel.STL" />
-      </geometry>
-      <material name="">
-        <color rgba="0.79216 0.81961 0.93333 1" />
-      </material>
-    </visual>
-    <collision>
-      <origin xyz="0 0 0" rpy="0 0 0" />
-      <geometry>
-        <mesh filename="file://$(find terrence_2)/description/meshes/DriverWheel.STL" />
+        <mesh filename="file://$(find description)/meshes/DriverWheel.STL" />
+      </geometry>
+      <material name="">
+        <color rgba="0.79216 0.81961 0.93333 1" />
+      </material>
+    </visual>
+    <collision>
+      <origin xyz="0 0 0" rpy="0 0 0" />
+      <geometry>
+        <mesh filename="file://$(find description)/meshes/DriverWheel.STL" />
       </geometry>
     </collision>
@@ -92,14 +92,14 @@
       <origin xyz="0 0 0" rpy="0 0 0" />
       <geometry>
-        <mesh filename="file://$(find terrence_2)/description/meshes/DriverSprocket.STL" />
-      </geometry>
-      <material name="">
-        <color rgba="0.79216 0.81961 0.93333 1" />
-      </material>
-    </visual>
-    <collision>
-      <origin xyz="0 0 0" rpy="0 0 0" />
-      <geometry>
-        <mesh filename="file://$(find terrence_2)/description/meshes/DriverSprocket.STL" />
+        <mesh filename="file://$(find description)/meshes/DriverSprocket.STL" />
+      </geometry>
+      <material name="">
+        <color rgba="0.79216 0.81961 0.93333 1" />
+      </material>
+    </visual>
+    <collision>
+      <origin xyz="0 0 0" rpy="0 0 0" />
+      <geometry>
+        <mesh filename="file://$(find description)/meshes/DriverSprocket.STL" />
       </geometry>
     </collision>
@@ -125,14 +125,14 @@
       <origin xyz="0 0 0" rpy="0 0 0" />
       <geometry>
-        <mesh filename="file://$(find terrence_2)/description/meshes/PassWheel.STL" />
-      </geometry>
-      <material name="">
-        <color rgba="0.79216 0.81961 0.93333 1" />
-      </material>
-    </visual>
-    <collision>
-      <origin xyz="0 0 0" rpy="0 0 0" />
-      <geometry>
-        <mesh filename="file://$(find terrence_2)/description/meshes/PassWheel.STL" />
+        <mesh filename="file://$(find description)/meshes/PassWheel.STL" />
+      </geometry>
+      <material name="">
+        <color rgba="0.79216 0.81961 0.93333 1" />
+      </material>
+    </visual>
+    <collision>
+      <origin xyz="0 0 0" rpy="0 0 0" />
+      <geometry>
+        <mesh filename="file://$(find description)/meshes/PassWheel.STL" />
       </geometry>
     </collision>
@@ -160,14 +160,14 @@
       <origin xyz="0 0 0" rpy="0 0 0" />
       <geometry>
-        <mesh filename="file://$(find terrence_2)/description/meshes/PassSprocket.STL" />
-      </geometry>
-      <material name="">
-        <color rgba="0.79216 0.81961 0.93333 1" />
-      </material>
-    </visual>
-    <collision>
-      <origin xyz="0 0 0" rpy="0 0 0" />
-      <geometry>
-        <mesh filename="file://$(find terrence_2)/description/meshes/PassSprocket.STL" />
+        <mesh filename="file://$(find description)/meshes/PassSprocket.STL" />
+      </geometry>
+      <material name="">
+        <color rgba="0.79216 0.81961 0.93333 1" />
+      </material>
+    </visual>
+    <collision>
+      <origin xyz="0 0 0" rpy="0 0 0" />
+      <geometry>
+        <mesh filename="file://$(find description)/meshes/PassSprocket.STL" />
       </geometry>
     </collision>
@@ -193,5 +193,5 @@
       <origin xyz="0 0 0" rpy="0 0 0" />
       <geometry>
-        <mesh filename="file://$(find terrence_2)/description/meshes/Loader.STL" />
+        <mesh filename="file://$(find description)/meshes/Loader.STL" />
       </geometry>
       <material name="">
@@ -202,5 +202,5 @@
       <origin xyz="0 0 0" rpy="0 0 0" />
       <geometry>
-        <mesh filename="file://$(find terrence_2)/description/meshes/Loader.STL" />
+        <mesh filename="file://$(find description)/meshes/Loader.STL" />
       </geometry>
     </collision>
@@ -228,14 +228,14 @@
       <origin xyz="0 0 0" rpy="0 0 0" />
       <geometry>
-        <mesh filename="file://$(find terrence_2)/description/meshes/Hopper.STL" />
-      </geometry>
-      <material name="">
-        <color rgba="0.79216 0.81961 0.93333 1" />
-      </material>
-    </visual>
-    <collision>
-      <origin xyz="0 0 0" rpy="0 0 0" />
-      <geometry>
-        <mesh filename="file://$(find terrence_2)/description/meshes/Hopper.STL" />
+        <mesh filename="file://$(find description)/meshes/Hopper.STL" />
+      </geometry>
+      <material name="">
+        <color rgba="0.79216 0.81961 0.93333 1" />
+      </material>
+    </visual>
+    <collision>
+      <origin xyz="0 0 0" rpy="0 0 0" />
+      <geometry>
+        <mesh filename="file://$(find description)/meshes/Hopper.STL" />
       </geometry>
     </collision>
@@ -261,14 +261,14 @@
       <origin xyz="0 0 0" rpy="0 0 0" />
       <geometry>
-        <mesh filename="file://$(find terrence_2)/description/meshes/Door.STL" />
-      </geometry>
-      <material name="">
-        <color rgba="0.79216 0.81961 0.93333 1" />
-      </material>
-    </visual>
-    <collision>
-      <origin xyz="0 0 0" rpy="0 0 0" />
-      <geometry>
-        <mesh filename="file://$(find terrence_2)/description/meshes/Door.STL" />
+        <mesh filename="file://$(find description)/meshes/Door.STL" />
+      </geometry>
+      <material name="">
+        <color rgba="0.79216 0.81961 0.93333 1" />
+      </material>
+    </visual>
+    <collision>
+      <origin xyz="0 0 0" rpy="0 0 0" />
+      <geometry>
+        <mesh filename="file://$(find description)/meshes/Door.STL" />
       </geometry>
     </collision>

Commit message: made the passive wheels mimic the sprockets in the urdf

File: ros2/description/urdf/ros2_control.xacro (robot description, xacro)
@@ -10,5 +10,5 @@
                 <param name="device">/dev/ttyACM0</param>
                 <param name="baud_rate">57600</param>
-                <param name="timeout_ms">1000</param>
+                <param name="timeout_ms">20</param>
             </hardware>
             <joint name="DS_Joint">

File: ros2/description/urdf/terrence.urdf.xacro (robot description, xacro)
@@ -76,4 +76,5 @@
     <axis xyz="1 0 0" />
     <limit effort="10" velocity="0" />
+    <mimic joint="DS_Joint" multiplier="1.0" offset="0.0"/>
   </joint>
   <gazebo reference="DriverWheel">
@@ -144,4 +145,5 @@
     <axis xyz="1 0 0" />
     <limit effort="10" velocity="0" />
+    <mimic joint="PS_Joint" multiplier="1.0" offset="0.0"/>
   </joint>
   <gazebo reference="PassWheel">

Commit message: commented out nonfunctional joints from real robot urdf

File: ros2/description/urdf/ros2_control.xacro (robot description, xacro)
@@ -28,5 +28,5 @@
                 <state_interface name="velocity"/>
             </joint>
-            <joint name="LoaderJoint">
+            <!-- <joint name="LoaderJoint">
                 <command_interface name="position"/>
                 <state_interface name="position"/>
@@ -39,5 +39,5 @@
             <joint name="DoorJoint">
                 <state_interface name="position"/>
-            </joint>
+            </joint> -->
         </ros2_control>
     </xacro:unless>

Commit message: added attachment logic to controller

File: ros2/description/urdf/ros2_control.xacro (robot description, xacro)
@@ -28,5 +28,5 @@
                 <state_interface name="velocity"/>
             </joint>
-            <!-- <joint name="LoaderJoint">
+            <joint name="LoaderJoint">
                 <command_interface name="position"/>
                 <state_interface name="position"/>
@@ -37,7 +37,4 @@
                 <state_interface name="position"/>
             </joint>
-            <joint name="DoorJoint">
-                <state_interface name="position"/>
-            </joint> -->
         </ros2_control>
     </xacro:unless>

Commit message: I would like to have a word with the creator of Gazebo harmonic. Also robot rotates about correct axis (no mimics). I also commented out cam in the URDF cuz it crashes GZ

File: ros2/description/urdf/ros2_control.xacro (robot description, xacro)
@@ -60,12 +60,4 @@
                 <state_interface name="position"/>
             </joint>
-            <joint name="DW_Joint">
-                <state_interface name="position"/>
-                <state_interface name="velocity"/>
-            </joint>
-            <joint name="PW_Joint">
-                <state_interface name="position"/>
-                <state_interface name="velocity"/>
-            </joint>
             <joint name="LoaderJoint">
                 <state_interface name="position"/>

File: ros2/description/urdf/terrence.urdf.xacro (robot description, xacro)
@@ -8,5 +8,5 @@
   <xacro:include filename="lidar.xacro"/>
   <!-- CAMERA -->
-  <xacro:include filename="camera.xacro"/>
+  <!-- <xacro:include filename="camera.xacro"/> -->
   <link name="base_link" />
   <link name="base_footprint" />
@@ -16,4 +16,5 @@
     <origin xyz="0 0 0" rpy="0 0 0" />
   </joint>
+  <!-- Base Link and Joint -->
   <link name="Base">
     <inertial>
@@ -50,5 +51,5 @@
     <inertial>
       <origin xyz="-0.030264 6.665E-05 1.2263E-10" rpy="0 0 0" />
-      <mass value="0.046607" />
+      <mass value="0.5" />
       <inertia ixx="3.7938E-05" ixy="-6.4305E-20" ixz="-1.3428E-19" iyy="1.9406E-05"
         iyz="2.6768E-13" izz="1.9256E-05" />
@@ -66,29 +67,69 @@
       <origin xyz="0 0 0" rpy="0 0 0" />
       <geometry>
-        <mesh filename="file://$(find description)/meshes/DriverWheel.STL" />
-      </geometry>
-    </collision>
-  </link>
-  <joint name="DW_Joint" type="continuous">
-    <origin xyz="0.17907 -0.0127 -0.0127" rpy="0 0 0" />
+        <!-- <mesh filename="file://$(find description)/meshes/DriverWheel.STL" /> -->
+        <sphere radius="0.05"/>
+      </geometry>
+    </collision>
+  </link>
+  <joint name="DW_Joint" type="fixed"> <origin xyz="0.17907 -0.0127 -0.0127" rpy="0 0 0" />
     <parent link="Base" />
     <child link="DriverWheel" />
-    <axis xyz="1 0 0" />
-    <limit effort="10" velocity="0" />
-    <mimic joint="DS_Joint" multiplier="1.0" offset="0.0"/>
   </joint>
   <gazebo reference="DriverWheel">
     <material>Gazebo/Blue</material>
-      <mu1 value="0.001"/>
-      <mu2 value="0.001"/>
+      <!-- <mu1 value="0.001"/>
+      <mu2 value="0.001"/> -->
+      <mu1 value="0.0"/>
+      <mu2 value="0.0"/>
+      <!-- <kp value="10000000.0" />
+      <kd value="1.0" /> -->
+  </gazebo>
+  <!-- Rear Caster Driver Wheel and Joint -->
+  <link name="RearDriverWheel">
+    <inertial>
+      <origin xyz="-0.030264 6.665E-05 1.2263E-10" rpy="0 0 0" />
+      <mass value="0.5" />
+      <inertia ixx="3.7938E-05" ixy="-6.4305E-20" ixz="-1.3428E-19" iyy="1.9406E-05"
+        iyz="2.6768E-13" izz="1.9256E-05" />
+    </inertial>
+    <!-- use sprocket for visual (it wont spin unfortunately) -->
+    <visual>
+      <origin xyz="-0.0397 0 0" rpy="0 0 0" />
+      <geometry>
+        <mesh filename="file://$(find description)/meshes/DriverSprocket.STL" />
+      </geometry>
+      <material name="blue">
+        <color rgba="0.79216 0.81961 0.93333 1" />
+      </material>
+    </visual>
+    <collision>
+      <origin xyz="-0.030264 6.665E-05 1.2263E-10" rpy="0 0 0" />
+      <geometry>
+        <!-- <mesh filename="file://$(find description)/meshes/DriverWheel.STL" /> -->
+        <sphere radius="0.05"/>
+      </geometry>
+    </collision>
+  </link>
+  <joint name="RDW_Joint" type="fixed"> <origin xyz="0.17907 -0.0127 -0.25959" rpy="0 0 0" />
+    <parent link="Base" />
+    <child link="RearDriverWheel" />
+  </joint>
+  <gazebo reference="RearDriverWheel">
+    <material>Gazebo/Pink</material>
+      <!-- <mu1 value="0.001"/>
+      <mu2 value="0.001"/> -->
+      <mu1 value="0.0"/>
+      <mu2 value="0.0"/>
+      <!-- <kp value="10000000.0" />
+      <kd value="1.0" /> -->
   </gazebo>
   <link name="DriverSprocket">
     <inertial>
       <origin xyz="0.0097746 -3.5292E-09 -5.2457E-08" rpy="0 0 0" />
-      <mass value="0.054042" />
+      <mass value="0.5" />
       <inertia ixx="5.3673E-05" ixy="-1.8152E-12" ixz="1.8049E-14" iyy="2.7245E-05"
         iyz="-1.9672E-11" izz="2.7245E-05" />
     </inertial>
-    <visual>
+    <!-- <visual>
       <origin xyz="0 0 0" rpy="0 0 0" />
       <geometry>
@@ -98,14 +139,15 @@
         <color rgba="0.79216 0.81961 0.93333 1" />
       </material>
-    </visual>
-    <collision>
-      <origin xyz="0 0 0" rpy="0 0 0" />
-      <geometry>
-        <mesh filename="file://$(find description)/meshes/DriverSprocket.STL" />
+    </visual> -->
+    <collision>
+      <origin xyz="0 0 0" rpy="0 0 0" />
+      <geometry>
+        <!-- <mesh filename="file://$(find description)/meshes/DriverSprocket.STL" /> -->
+        <sphere radius="0.05"/>
       </geometry>
     </collision>
   </link>
   <joint name="DS_Joint" type="continuous">
-    <origin xyz="0.14605 -0.012431 -0.25959" rpy="0 0 0" />
+    <origin xyz="0.14605 -0.0127 -0.136145" rpy="0 0 0" />
     <parent link="Base" />
     <child link="DriverSprocket" />
@@ -119,5 +161,5 @@
     <inertial>
       <origin xyz="0.020612 8.4006E-05 -0.00023239" rpy="0 0 0" />
-      <mass value="0.046607" />
+      <mass value="0.5" />
       <inertia ixx="3.7938E-05" ixy="-6.4876E-20" ixz="-1.3466E-19" iyy="1.9406E-05"
         iyz="-3.2644E-10" izz="1.9256E-05" />
@@ -135,29 +177,61 @@
       <origin xyz="0 0 0" rpy="0 0 0" />
       <geometry>
-        <mesh filename="file://$(find description)/meshes/PassWheel.STL" />
-      </geometry>
-    </collision>
-  </link>
-  <joint name="PW_Joint" type="continuous">
-    <origin xyz="-0.17907 -0.0127 -0.0127" rpy="0 0 0" />
+        <!-- <mesh filename="file://$(find description)/meshes/PassWheel.STL" /> -->
+        <sphere radius="0.05"/>
+      </geometry>
+    </collision>
+  </link>
+  <joint name="PW_Joint" type="fixed"> <origin xyz="-0.17907 -0.0127 -0.0127" rpy="0 0 0" />
     <parent link="Base" />
     <child link="PassWheel" />
-    <axis xyz="1 0 0" />
-    <limit effort="10" velocity="0" />
-    <mimic joint="PS_Joint" multiplier="1.0" offset="0.0"/>
   </joint>
   <gazebo reference="PassWheel">
     <material>Gazebo/Blue</material>
-      <mu1 value="0.001"/>
-      <mu2 value="0.001"/>
+      <mu1 value="0.0"/>
+      <mu2 value="0.0"/>
+  </gazebo>
+  <!-- rear pass wheel -->
+  <link name="RearPassWheel">
+    <inertial>
+      <origin xyz="0.020612 8.4006E-05 -0.00023239" rpy="0 0 0" />
+      <mass value="0.5" />
+      <inertia ixx="3.7938E-05" ixy="-6.4876E-20" ixz="-1.3466E-19" iyy="1.9406E-05"
+        iyz="-3.2644E-10" izz="1.9256E-05" />
+    </inertial>
+    <!-- sprocket visual - again, it wont move -->
+    <visual>
+      <origin xyz="0.0397 0 0" rpy="0 0 0" />
+      <geometry>
+        <mesh filename="file://$(find description)/meshes/PassSprocket.STL" />
+      </geometry>
+      <material name="gray">
+        <color rgba="0.79216 0.81961 0.93333 1" />
+      </material>
+    </visual>
+    <collision>
+      <origin xyz="0.020612 8.4006E-05 -0.00023239" rpy="0 0 0" />
+      <geometry>
+        <!-- <mesh filename="file://$(find description)/meshes/PassWheel.STL" /> -->
+        <sphere radius="0.05"/>
+      </geometry>
+    </collision>
+  </link>
+  <joint name="RPW_Joint" type="fixed"> <origin xyz="-0.17907 -0.0127 -0.25959" rpy="0 0 0" />
+    <parent link="Base" />
+    <child link="RearPassWheel" />
+  </joint>
+  <gazebo reference="RearPassWheel">
+    <material>Gazebo/White</material>
+      <mu1 value="0.0"/>
+      <mu2 value="0.0"/>
   </gazebo>
   <link name="PassSprocket">
     <inertial>
       <origin xyz="-0.0056813 -3.6211E-09 -5.2434E-08" rpy="0 0 0" />
-      <mass value="0.054042" />
+      <mass value="0.5" />
       <inertia ixx="5.3673E-05" ixy="-1.8152E-12" ixz="2.2008E-14" iyy="2.7245E-05"
         iyz="-2.0018E-11" izz="2.7245E-05" />
     </inertial>
-    <visual>
+    <!-- <visual>
       <origin xyz="0 0 0" rpy="0 0 0" />
       <geometry>
@@ -167,14 +241,15 @@
         <color rgba="0.79216 0.81961 0.93333 1" />
       </material>
-    </visual>
-    <collision>
-      <origin xyz="0 0 0" rpy="0 0 0" />
-      <geometry>
-        <mesh filename="file://$(find description)/meshes/PassSprocket.STL" />
+    </visual> -->
+    <collision>
+      <origin xyz="0 0 0" rpy="0 0 0" />
+      <geometry>
+        <!-- <mesh filename="file://$(find description)/meshes/PassSprocket.STL" /> -->
+        <sphere radius="0.05"/>
       </geometry>
     </collision>
   </link>
   <joint name="PS_Joint" type="continuous">
-    <origin xyz="-0.14605 -0.012969 -0.25959" rpy="0 0 0" />
+    <origin xyz="-0.14605 -0.0127 -0.136145" rpy="0 0 0" />
     <parent link="Base" />
     <child link="PassSprocket" />
@@ -286,3 +361,14 @@
     <material>Gazebo/White</material>
   </gazebo>
+  <!-- Mimic joints -->
+  <!-- <gazebo>
+    <plugin filename="gz-sim-mimic-joint-system" name="gz::sim::systems::MimicJoint">
+        <joint>DS_Joint</joint>
+        <mimicJoint>DW_Joint</mimicJoint>
+    </plugin>
+    <plugin filename="gz-sim-mimic-joint-system" name="gz::sim::systems::MimicJoint">
+        <joint>PS_Joint</joint>
+        <mimicJoint>PW_Joint</mimicJoint>
+    </plugin>
+  </gazebo> -->
 </robot>
