Commit message: Fixed costmap. Converted DepthCloud to PointCloud on depth camera

File: ros2/description/urdf/camera.xacro (robot description, xacro)
@@ -25,5 +25,5 @@
         <parent link="camera_link"/>
         <child link="camera_link_optical"/>
-        <origin xyz="0.1 0 0" rpy="${-pi/2} 0 ${-pi/2}"/>
+        <origin xyz="0.1 0 0" rpy="0 0 0"/>
     </joint>
     <link name="camera_link_optical"></link>
